File: Alpha-13/Transmitter and Receiver Module/Receiver Schematics.sch (EAGLE design)
At the start: 3 parts, among them M1 WIRELESS-XY-MK-5V

Commit message: Codes nd Details
Connections:
- net N$4: now also PCB1.5V; no longer PCB1.3.3V
Changed lines of the file:
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@@
 <wire x1="10.16" y1="66.04" x2="15.24" y2="66.04" width="0.1524" layer="91"/>
 <wire x1="15.24" y1="66.04" x2="15.24" y2="35.56" width="0.1524" layer="91"/>
-<wire x1="15.24" y1="35.56" x2="48.26" y2="35.56" width="0.1524" layer="91"/>
-<pinref part="PCB1" gate="G$1" pin="3.3V"/>
-<wire x1="48.26" y1="35.56" x2="48.26" y2="40.64" width="0.1524" layer="91"/>
+<wire x1="15.24" y1="35.56" x2="50.8" y2="35.56" width="0.1524" layer="91"/>
+<pinref part="PCB1" gate="G$1" pin="5V"/>
+<wire x1="50.8" y1="40.64" x2="50.8" y2="35.56" width="0.1524" layer="91"/>
 </segment>
 </net>
